File: steuerung_automatik/hardware/kicad_dezentral/filament_dryer.kicad_pcb (KiCad board)
At the start: 2 copper layers, 94 x 130 mm, 136 parts, among them J1 USB_C_Receptacle_USB2.0, J2 H/T Ambient, J3 T Aux, J4 Peristaltic Pump, Q3 NMOS, Q4 NMOS, Q5 NMOS, Q6 NMOS, Q7 NMOS, Q8 NMOS, U1 W25Q128JVS, U2 AMS1117-3.3, U3 RP2040, U4 DS18B20Z, U5 H/T Filament, X1 12MHz Yangxing Tech X322512MS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

Commit message: Update components
Parts:
- removed C17, C18: 30p, Capacitor_SMD:C_0402_1005Metric
- removed C20: 10u, Capacitor_SMD:C_0603_1608Metric
- removed D2: General Purpose Diode, 00_project_library:D_SMA
- removed D3: POW_LED, 00_project_library:LED_0603_1608Metric
- removed D6: FAN_1, 00_project_library:LED_0603_1608Metric
- removed D7: FAN_2, 00_project_library:LED_0603_1608Metric
- removed H5: MountingHole, MountingHole:MountingHole_3.2mm_M3
- removed J2: H/T Ambient, 00_project_library:grove_vert_holes
- removed J3: T Aux, 00_project_library:grove_vert_holes
- removed J4: Peristaltic Pump, 00_project_library:grove_vert_holes
- removed JP1, JP2, JP3, JP4: SolderJumper_2_Open, Jumper:SolderJumper-2_P1.3mm_Open_RoundedPad1.0x1.5mm
- removed NeoC1, NeoC10, NeoC11, NeoC12, NeoC13, NeoC14, NeoC15, NeoC16, NeoC17, NeoC18, NeoC19, NeoC2, NeoC20, NeoC21, NeoC22, NeoC23, NeoC24, NeoC25, NeoC26, NeoC27, NeoC28, NeoC3, NeoC4, NeoC5, NeoC6, NeoC7, NeoC8, NeoC9: 100n, Capacitor_SMD:C_0402_1005Metric_Pad0.74x0.62mm_HandSolder
- removed NeoD1, NeoD10, NeoD11, NeoD12, NeoD13, NeoD14, NeoD15, NeoD16, NeoD17, NeoD18, NeoD19, NeoD2, NeoD20, NeoD21, NeoD22, NeoD23, NeoD24, NeoD25, NeoD26, NeoD27, NeoD28, NeoD3, NeoD4, NeoD5, NeoD6, NeoD7, NeoD8, NeoD9: WS2812B-2020, LED_SMD:LED_WS2812B-2020_PLCC4_2.0x2.0mm
- removed Q3, Q4, Q5, Q6, Q7, Q8: NMOS, 00_project_library:SOT-23
- removed R10: 1k, Resistor_SMD:R_0402_1005Metric_Pad0.72x0.64mm_HandSolder
- removed R12, R13, R14: 10k, Resistor_SMD:R_0402_1005Metric_Pad0.72x0.64mm_HandSolder
- removed R15, R16: 4k7, Resistor_SMD:R_0402_1005Metric_Pad0.72x0.64mm_HandSolder
- removed R17, R18, R21: 4K7, Resistor_SMD:R_0402_1005Metric_Pad0.72x0.64mm_HandSolder
- removed R19, R20, R22: 470R, Resistor_SMD:R_0402_1005Metric_Pad0.72x0.64mm_HandSolder
- removed R9: 10K, Resistor_SMD:R_0402_1005Metric_Pad0.72x0.64mm_HandSolder
- removed SW_BOOT1: Boot, 00_project_library:SW_TS-1187A-B-A-B
- removed SW_RESET1: Reset, 00_project_library:SW_TS-1187A-B-A-B
- removed TP10: FAN_SILICAGEL_GND, TestPoint:TestPoint_Pad_D3.0mm
- removed TP11: HT_SILICAGEL_SCL, TestPoint:TestPoint_Pad_D3.0mm
- removed TP2: HT_SILICAGEL_GND, TestPoint:TestPoint_Pad_D3.0mm
- removed TP3: HT_SILICAGEL_3V3, TestPoint:TestPoint_Pad_D3.0mm
- removed TP6: HT_SILICAGEL_SCA, TestPoint:TestPoint_Pad_D3.0mm
- removed TP7: FAN_AMBIENT_5V, TestPoint:TestPoint_Pad_D3.0mm
- removed TP8: FAN_AMBIENT_GND, TestPoint:TestPoint_Pad_D3.0mm
- removed TP9: FAN_SILICAGEL_5V, TestPoint:TestPoint_Pad_D3.0mm
- removed U4: DS18B20Z, 00_project_library:SOIC-8_3.9x4.9mm_P1.27mm
- removed U5: H/T Filament, 00_project_library:SON50P250X250X90-9T110X180N
- removed X1: 12MHz Yangxing Tech X322512MSB4SI, 00_project_library:Crystal_SMD_3225-4Pin_3.2x2.5mm
- removed dryer_print3D1: dryer_print3D, 00_project_library:dryer_print3d
- added C16: 10u, Capacitor_SMD:C_0603_1608Metric, F.Cu at (128.6, 72.7)
- added R7: 10K, Resistor_SMD:R_0402_1005Metric_Pad0.72x0.64mm_HandSolder, F.Cu at (106.1, 73.6)
- added SW1: SW_MEC_5E, 00_project_library:SW_TS-1187A-B-A-B, F.Cu at (112.6, 64.0)
- added SW2: SW_MEC_5E, 00_project_library:SW_TS-1187A-B-A-B, F.Cu at (112.6, 70.7)
- added Y1: Crystal_GND24_Small, 00_project_library:Crystal_SMD_3225-4Pin_3.2x2.5mm, F.Cu at (128.8, 79.1)
- C13, C14: value 10u -> 100n; footprint Capacitor_SMD:C_0603_1608Metric -> Capacitor_SMD:C_0402_1005Metric_Pad0.74x0.62mm_HandSolder
- C3: value 100n -> 1u
- C5: value 1u -> 100n
- C7, C8: value 100n -> 30p; footprint Capacitor_SMD:C_0402_1005Metric_Pad0.74x0.62mm_HandSolder -> Capacitor_SMD:C_0402_1005Metric
- D1: value General Purpose Diode -> LED GREEN; footprint 00_project_library:D_SMA -> 00_project_library:LED_0603_1608Metric
- R1: value 4K7 -> 5.1K
- R2: value 10K -> 5.1K
- R3, R4: value 5.1K -> 27R
- R5: value 27R -> 10K
- R6: value 27R -> 470R
- R8: value 470R -> 1k
- U1: value W25Q128JVS -> RP2040; footprint 00_project_library:SOIC-8_5.23x5.23mm_P1.27mm -> Package_DFN_QFN:QFN-56-1EP_7x7mm_P0.4mm_EP5.6x5.6mm
- U2: value AMS1117-3.3 -> W25Q128JVS; footprint 00_project_library:SOT-223-3_TabPin2 -> 00_project_library:SOIC-8_5.23x5.23mm_P1.27mm
- U3: value RP2040 -> AMS1117-3.3; footprint 00_project_library_circuitstate:RP2040-QFN-56 -> Package_TO_SOT_SMD:SOT-223-3_TabPin2
- moved D1 81.7 mm to (128.6, 75.3), turned to 0 degrees
- moved C14 70.0 mm to (124.9, 75.9)
- moved R1 59.7 mm to (106.1, 61.7), turned to 0 degrees
- moved TP1 50.5 mm to (128.5, 83.6)
- moved C13 38.8 mm to (124.9, 73.9), turned to 0 degrees
- moved R8 33.9 mm to (106.1, 75.6), turned to 0 degrees
- moved U1 33.8 mm to (121.6, 81.5), turned to 0 degrees
- moved C15 33.7 mm to (128.6, 70.2), turned to 0 degrees
- moved C11 28.2 mm to (124.9, 69.9), turned to 0 degrees
- moved U2 25.5 mm to (111.1, 79.2), turned to 0 degrees
- moved C1 25.3 mm to (118.5, 69.9), turned to 0 degrees
- moved C8 22.3 mm to (128.2, 63.7)
- moved C7 21.1 mm to (128.2, 61.7)
- moved U3 20.6 mm to (121.8, 64.8)
- moved C4 20.2 mm to (118.5, 75.9), turned to 0 degrees
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Connections:
- C1 pad 1: +3V3 -> +1V1
- C13 pad 1: +5V -> +3V3
- C15 pad 1: +3V3 -> +5V
- C4 pad 1: +1V1 -> +3V3
- C7 pad 1: +3V3 -> /XIN
- C8 pad 1: +3V3 -> Net-(C8-Pad1)
- D1 pad 1: +5V -> Net-(D1-K)
- D1 pad 2: Net-(D1-A) -> +3V3
- R1 pad 1: +5V -> Net-(J1-CC1)
- R1 pad 2: Net-(JP1-B) -> GND
- R2 pad 1: +3V3 -> Net-(J1-CC2)
- R2 pad 2: /QSPI_SS -> GND
- R3 pad 1: Net-(J1-CC1) -> /USB_D+
- R3 pad 2: GND -> Net-(U1-USB-DP)
- R4 pad 1: Net-(J1-CC2) -> /USB_D-
- R4 pad 2: GND -> Net-(U1-USB-DM)
- R5 pad 1: /USB_D+ -> +3V3
- R5 pad 2: Net-(U3-USB-DP) -> /RUN
- R6 pad 1: /USB_D- -> GND
- R6 pad 2: Net-(U3-USB-DM) -> Net-(D1-K)
- R8 pad 1: GND -> /XOUT
- R8 pad 2: Net-(D3-K) -> Net-(C8-Pad1)
- U1 pad 1: /QSPI_SS -> +3V3
- U1 pad 2: /QSPI_SD1 -> unconnected-(U1-GPIO0-Pad2)
- U1 pad 3: /QSPI_SD2 -> unconnected-(U1-GPIO1-Pad3)
- U1 pad 4: GND -> unconnected-(U1-GPIO2-Pad4)
- U1 pad 5: /QSPI_SD0 -> unconnected-(U1-GPIO3-Pad5)
- U1 pad 6: /QSPI_SCLK -> unconnected-(U1-GPIO4-Pad6)
- U1 pad 7: /QSPI_SD3 -> unconnected-(U1-GPIO5-Pad7)
- U1 pad 8: +3V3 -> unconnected-(U1-GPIO6-Pad8)
- U2 pad 1: GND -> /QSPI_SS
- U2 pad 2: +3V3 -> /QSPI_SD1
- U2 pad 3: +5V -> /QSPI_SD2
- U3 pad 1: +3V3 -> GND
- U3 pad 2: /GPIO_NP_BOARD -> +3V3
- U3 pad 3: /GPIO_NP_A -> +5V
Routing:
- net +3V3: track 424.0 -> 0.00 mm, vias 14 -> 0
- net +5V: track 295.0 -> 0.00 mm, vias 2 -> 0
- net GND: track 189.3 -> 10.8 mm, vias 109 -> 0
- net /HT_BOARD_SCL: track 117.2 -> 0.00 mm, vias 4 -> 0
- net /GPIO_FAN_AMBIENT: track 107.5 -> 0.00 mm, vias 4 -> 0
- net /HT_BOARD_SDA: track 107.3 -> 0.00 mm, vias 3 -> 0
- net /GPIO_FAN_SILICAGEL: track 99.2 -> 0.00 mm, vias 2 -> 0
- net Net-(JP2-B): track 91.1 -> 0.00 mm
- net /T_HEATING_1WIRE: track 90.4 -> 0.00 mm, vias 3 -> 0
- net Net-(JP1-B): track 79.2 -> 0.00 mm
- net Net-(JP3-B): track 64.4 -> 0.00 mm
- net /RUN: track 54.6 -> 0.00 mm, vias 2 -> 0
- net /GPIO_NP_BOARD: track 48.2 -> 0.00 mm
- net /QSPI_SS: track 38.3 -> 0.00 mm
- net /GPIO_NP_B: track 35.8 -> 0.00 mm, vias 2 -> 0
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- removed copper zone on F.Cu, net +5V
Other:
- board outline removed
- board text removed: "*"
- board text removed: "RP2040"
