File: steuerung_automatik/hardware/kicad_dezentral/filament_dryer.kicad_sch (KiCad schematic)
At the start: 136 parts, among them J1 USB_C_Receptacle_USB2.0, J2 H/T Ambient, J3 T Aux, J4 Peristaltic Pump, Q3 NMOS, Q4 NMOS, Q5 NMOS, Q6 NMOS, Q7 NMOS, Q8 NMOS, U1 W25Q128JVS, U2 AMS1117-3.3, U3 RP2040, U4 DS18B20Z, U5 H/T Filament, X1 12MHz Yangxing Tech X322512MS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

Commit message: Update components
Parts:
- removed C14, C20: 10u, Capacitor_SMD:C_0603_1608Metric, symbol 00_project_library:C
- removed D1, D2: General Purpose Diode, 00_project_library:D_SMA, symbol 00_project_library:GeneralPurposeDiode
- removed D6: FAN_1, 00_project_library:LED_0603_1608Metric, symbol 00_project_library:LED
- removed D7: FAN_2, 00_project_library:LED_0603_1608Metric, symbol 00_project_library:LED
- removed H5: MountingHole, MountingHole:MountingHole_3.2mm_M3, symbol 00_project_library:MountingHole
- removed J2: H/T Ambient, 00_project_library:grove_vert_holes, symbol 00_project_library:grove_vert_holes_1
- removed J3: T Aux, 00_project_library:grove_vert_holes, symbol 00_project_library:grove_vert_holes
- removed J4: Peristaltic Pump, 00_project_library:grove_vert_holes, symbol 00_project_library:grove_vert_holes
- removed JP1, JP2, JP3, JP4: SolderJumper_2_Open, Jumper:SolderJumper-2_P1.3mm_Open_RoundedPad1.0x1.5mm, symbol Jumper:SolderJumper_2_Open
- removed NeoC1, NeoC10, NeoC11, NeoC12, NeoC13, NeoC14, NeoC15, NeoC16, NeoC17, NeoC18, NeoC19, NeoC2, NeoC20, NeoC21, NeoC22, NeoC23, NeoC24, NeoC25, NeoC26, NeoC27, NeoC28, NeoC3, NeoC4, NeoC5, NeoC6, NeoC7, NeoC8, NeoC9: 100n, Capacitor_SMD:C_0402_1005Metric_Pad0.74x0.62mm_HandSolder, symbol 00_project_library:C
- removed NeoD1, NeoD10, NeoD11, NeoD12, NeoD13, NeoD14, NeoD15, NeoD16, NeoD17, NeoD18, NeoD19, NeoD2, NeoD20, NeoD21, NeoD22, NeoD23, NeoD24, NeoD25, NeoD26, NeoD27, NeoD28, NeoD3, NeoD4, NeoD5, NeoD6, NeoD7, NeoD8, NeoD9: WS2812B-2020, LED_SMD:LED_WS2812B-2020_PLCC4_2.0x2.0mm, symbol 00_project_library:WS2812B-2020
- removed Q3, Q4, Q5, Q6, Q7, Q8: NMOS, 00_project_library:SOT-23, symbol 00_project_library:NMOS
- removed R1, R17, R18, R21: 4K7, Resistor_SMD:R_0402_1005Metric_Pad0.72x0.64mm_HandSolder, symbol 00_project_library:R
- removed R12, R13, R14: 10k, Resistor_SMD:R_0402_1005Metric_Pad0.72x0.64mm_HandSolder, symbol 00_project_library:R
- removed R15, R16: 4k7, Resistor_SMD:R_0402_1005Metric_Pad0.72x0.64mm_HandSolder, symbol 00_project_library:R
- removed R19, R20, R22: 470R, Resistor_SMD:R_0402_1005Metric_Pad0.72x0.64mm_HandSolder, symbol 00_project_library:R
- removed TP10: FAN_SILICAGEL_GND, TestPoint:TestPoint_Pad_D3.0mm, symbol Connector:TestPoint
- removed TP11: HT_SILICAGEL_SCL, TestPoint:TestPoint_Pad_D3.0mm, symbol Connector:TestPoint
- removed TP2: HT_SILICAGEL_GND, TestPoint:TestPoint_Pad_D3.0mm, symbol Connector:TestPoint
- removed TP3: HT_SILICAGEL_3V3, TestPoint:TestPoint_Pad_D3.0mm, symbol Connector:TestPoint
- removed TP6: HT_SILICAGEL_SCA, TestPoint:TestPoint_Pad_D3.0mm, symbol Connector:TestPoint
- removed TP7: FAN_AMBIENT_5V, TestPoint:TestPoint_Pad_D3.0mm, symbol Connector:TestPoint
- removed TP8: FAN_AMBIENT_GND, TestPoint:TestPoint_Pad_D3.0mm, symbol Connector:TestPoint
- removed TP9: FAN_SILICAGEL_5V, TestPoint:TestPoint_Pad_D3.0mm, symbol Connector:TestPoint
- removed U4: DS18B20Z, 00_project_library:SOIC-8_3.9x4.9mm_P1.27mm, symbol 00_project_library:DS18B20Z
- removed U5: H/T Filament, 00_project_library:SON50P250X250X90-9T110X180N, symbol 00_project_library:SHT31-DIS
- removed dryer_print3D1: dryer_print3D, 00_project_library:dryer_print3d, symbol 00_project_library:dryer_print3d
- D1: renamed from D3; value POW_LED -> LED GREEN; symbol 00_project_library:LED -> 00_project_library:LED GREEN; JLC C2290 -> C2297
- J1: Digikey (none) -> https://www.digikey.com/en/products/detail/gct/USB4105-GF-A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
- R1: renamed from R3; symbol 00_project_library:R_Small -> Device:R
- R2: renamed from R4; symbol 00_project_library:R_Small -> Device:R
- R3: renamed from R5; symbol 00_project_library:R -> Device:R
- R4: renamed from R6; symbol 00_project_library:R -> Device:R
- R5: renamed from R9; symbol 00_project_library:R -> Device:R
- R6: renamed from R8; symbol 00_project_library:R -> Device:R
- R7: renamed from R2; symbol 00_project_library:R -> Device:R
- R8: renamed from R10; symbol 00_project_library:R -> Device:R
- SW1: renamed from SW_RESET1; value Reset -> SW_MEC_5E
- SW2: renamed from SW_BOOT1; value Boot -> SW_MEC_5E
- U1: renamed from U3; footprint 00_project_library_circuitstate:RP2040-QFN-56 -> Package_DFN_QFN:QFN-56-1EP_7x7mm_P0.4mm_EP5.6x5.6mm; JLC (none) -> C2040
- U2: renamed from U1; JLC (none) -> C97521
- U3: renamed from U2; footprint 00_project_library:SOT-223-3_TabPin2 -> Package_TO_SOT_SMD:SOT-223-3_TabPin2; symbol Regulator_Linear:AMS1117-3.3 -> 00_project_library:AMS1117-3.3
- Y1: renamed from X1; value 12MHz Yangxing Tech X322512MSB4SI -> Crystal_GND24_Small
- renumbered C2 to C1, C9 to C10, C10 to C11, C11 to C12, C12 to C13, C1 to C14, C13 to C15, C15 to C16, C3 to C2, C4 to C3, C5 to C4, C6 to C5, C7 to C6, C17 to C7, C18 to C8, C8 to C9
Connections:
- net GPIO_FAN_AMBIENT: no longer names the net of U1.32 (GPIO21)
- net GPIO_FAN_SILICAGEL: no longer names the net of U1.12 (GPIO9)
- net GPIO_NP_A: no longer names the net of U1.3 (GPIO1)
- net GPIO_NP_B: no longer names the net of U1.37 (GPIO25)
- net GPIO_NP_BOARD: no longer names the net of U1.2 (GPIO0)
- net GPIO_NP_C: no longer names the net of U1.4 (GPIO2)
- net GPIO_PUMP_STEP: no longer names the net of U1.27 (GPIO16)
- net HT_BOARD_SCL: no longer names the net of U1.39 (GPIO27/ADC1)
- net HT_BOARD_SDA: no longer names the net of U1.38 (GPIO26/ADC0)
- net HT_GROVE_SCL: no longer names the net of U1.16 (GPIO13)
- net HT_GROVE_SDA: no longer names the net of U1.15 (GPIO12)
- net T_AUX_1WIRE: no longer names the net of U1.17 (GPIO14)
- net T_HEATING_1WIRE: no longer names the net of U1.18 (GPIO15)
- no-connect marks 28 -> 34
Other:
- note removed: "Fan Ambient"
- note removed: "Fan Silicagel"
- note removed: "H/T Ambient I2C0 0x44"
- note removed: "H/T Filament I2C1 0x45"
- note removed: "H/T Silicagel I2C1 0x44"
- note removed: "Neopixel WS2812B-2020"
- note removed: "Peristaltic Pump"
- note removed: "Temperature"
- note removed: "print3D"
- moved on the sheet: H1, H2, H3, H4
