File: steuerung_automatik/hardware/pcb_kicad/pcb_zentral_haus.kicad_sch (KiCad schematic)
At the start: 9 parts, among them U301 SP3485EN-L/TR

Commit message: Nach Review
Parts:
- added D301: LED GREEN, 00_project_library:LED_0603_1608Metric, symbol 00_project_library:LED GREEN
- added D302: LED WHITE, 00_project_library:LED_0603_1608Metric, symbol 00_project_library:LED WHITE
- added R302: 470, Resistor_SMD:R_0805_2012Metric, symbol 00_project_circuitstate-obsolete:R
- R301: value 1K -> 470
- renumbered D301 to D303, D302 to D304, D303 to D305, R302 to R303, R303 to R304, R304 to R305
Connections:
- net +3V3: now also R303.1, D301.2 (A); no longer R305.2
- net A: no longer D303.1 (A1), D304.2 (A2), R303.2, R304.1, U301.6 (A)
- net B: no longer D304.1 (A1), D305.2 (A2), R304.2, R305.1, U301.7 (B)
- net ENABLE: no longer U301.2 (~{RE}), U301.3 (DE)
- net GND: now also R305.2, R302.2; no longer R303.1
- net MODBUS_RO: now also U301.1 (RO); no longer R301.1
- net MODBUS_RE: now reaches R301.2
- net MODBUS_RE: now also Haus301.7 (MODBUS_RE), U301.2 (~{RE}); no longer U301.1 (RO)
- new net: D302.1 (K), R302.1
- new net: D301.1 (K), R301.1
- new net 485_A: D303.1 (A1), D304.2 (A2), R303.2, R304.1, U301.6 (A)
- new net 485_B: D304.1 (A1), D305.2 (A2), R304.2, R305.1, U301.7 (B)
- new net MODBUS_DE: D302.2 (A), Haus301.8 (MODBUS_DE), U301.3 (DE)
