File: steuerung_automatik/hardware/pcb_kicad/pcb_zentral_pi.kicad_pcb (KiCad board)
At the start: 2 copper layers, 40 parts, among them J1 USB_C_Receptacle_USB2.0, J2 weidmueller_SL 5.08HC-04-180, J3 weidmueller_SL 5.08HC-12-180, SW1 SW_MEC_5E, SW2 SW_MEC_5E, U1 RP2040, U2 W25Q128JVS, U3 AMS1117-3.3, U4 SP3485EN-L/TR, Y1 Crystal_GND24_Small

Commit message: Vor Review
Parts:
- removed C1, C10, C11, C12, C13, C14, C2, C5, C6, C9: 100n, Capacitor_SMD:C_0402_1005Metric_Pad0.74x0.62mm_HandSolder
- removed C15, C16: 10u, Capacitor_SMD:C_0603_1608Metric
- removed C3, C4: 1u, Capacitor_SMD:C_0402_1005Metric_Pad0.74x0.62mm_HandSolder
- removed C7, C8: 30p, Capacitor_SMD:C_0402_1005Metric
- removed D1: LED GREEN, 00_project_library:LED_0603_1608Metric
- removed H1, H2, H3, H4: MountingHole, MountingHole:MountingHole_3.2mm_M3
- removed J1: USB_C_Receptacle_USB2.0, 00_project_library:USB_C_Receptacle_Palconn_UTC16-G
- removed J2: weidmueller_SL 5.08HC-04-180, 00_project_library:weidmueller_SL 5.08HC-04-180
- removed J3: weidmueller_SL 5.08HC-12-180, 00_project_library:weidmueller_SL 5.08HC-12-180
- removed R1, R2: 5.1K, Resistor_SMD:R_0402_1005Metric_Pad0.72x0.64mm_HandSolder
- removed R3, R4: 27R, Resistor_SMD:R_0402_1005Metric_Pad0.72x0.64mm_HandSolder
- removed R5, R7: 10K, Resistor_SMD:R_0402_1005Metric_Pad0.72x0.64mm_HandSolder
- removed R6: 470R, Resistor_SMD:R_0402_1005Metric_Pad0.72x0.64mm_HandSolder
- removed R8: 1k, Resistor_SMD:R_0402_1005Metric_Pad0.72x0.64mm_HandSolder
- removed SW1, SW2: SW_MEC_5E, 00_project_library:SW_TS-1187A-B-A-B
- removed TP1: TestPoint, TestPoint:TestPoint_Pad_D2.5mm
- removed U1: RP2040, 00_project_library:RP2040-QFN-56
- removed U2: W25Q128JVS, 00_project_library:SOIC-8_5.23x5.23mm_P1.27mm
- removed U3: AMS1117-3.3, 00_project_library:SOT-223-3_TabPin2
- removed U4: SP3485EN-L/TR, Package_SO:SOIC-8_3.9x4.9mm_P1.27mm
- removed Y1: Crystal_GND24_Small, 00_project_library:Crystal_SMD_3225-4Pin_3.2x2.5mm
- added D301: SMAJ6.5CA, Diode_SMD:D_SMA, F.Cu at (148.6, 165.2)
- added D302: SMAJ6.5CA, Diode_SMD:D_SMA, F.Cu at (144.9, 170.7)
- added D303: SMAJ6.5CA, Diode_SMD:D_SMA, F.Cu at (142.4, 165.2)
- added D401: SMAJ6.5CA, Diode_SMD:D_SMA, F.Cu at (158.8, 165.2)
- added D402: SMAJ6.5CA, Diode_SMD:D_SMA, F.Cu at (155.1, 170.7)
- added D403: SMAJ6.5CA, Diode_SMD:D_SMA, F.Cu at (152.5, 165.2)
- added D501: SMAJ6.5CA, Diode_SMD:D_SMA, F.Cu at (168.9, 165.2)
- added D502: SMAJ6.5CA, Diode_SMD:D_SMA, F.Cu at (165.2, 170.7)
- added D503: SMAJ6.5CA, Diode_SMD:D_SMA, F.Cu at (162.7, 165.2)
- added D601: SMAJ6.5CA, Diode_SMD:D_SMA, F.Cu at (179.1, 165.2)
- added D602: SMAJ6.5CA, Diode_SMD:D_SMA, F.Cu at (175.4, 170.7)
- added D603: SMAJ6.5CA, Diode_SMD:D_SMA, F.Cu at (172.9, 165.2)
- added H101: MountingHole, MountingHole:MountingHole_3.2mm_M3, F.Cu at (68.8, 3.48)
- added H102: MountingHole, MountingHole:MountingHole_3.2mm_M3, F.Cu at (68.8, 11.4)
- added H103: MountingHole, MountingHole:MountingHole_3.2mm_M3, F.Cu at (68.8, 19.4)
- added H104: MountingHole, MountingHole:MountingHole_3.2mm_M3, F.Cu at (68.8, 27.3)
- added Haus201: floor_Hausreihe, 00_project_library:floor_Hausreihe, F.Cu at (183.0, 133.7)
- added Haus301: ~, 00_project_library:floor_Haus, F.Cu at (150.4, 177.6)
- added Haus401: ~, 00_project_library:floor_Haus, F.Cu at (160.6, 177.6)
- added Haus501: ~, 00_project_library:floor_Haus, F.Cu at (170.8, 177.6)
- added Haus601: ~, 00_project_library:floor_Haus, F.Cu at (180.9, 177.6)
- added J101: pi_zero, 00_project_library:rpi_zero_bottom, F.Cu at (153.6, 68.3)
- added J201: weidmueller_SL5.08HC-12-90, 00_project_library:weidmueller_SL5.08HC-12-90, F.Cu at (122.7, 181.6)
- added R301: 1K, Resistor_SMD:R_0805_2012Metric, F.Cu at (143.5, 151.1)
- added R302: 4K7, Resistor_SMD:R_0805_2012Metric, F.Cu at (147.2, 173.5)
- added R303: 120, Resistor_SMD:R_0805_2012Metric, F.Cu at (143.2, 173.5)
- added R304: 4K7, Resistor_SMD:R_0805_2012Metric, F.Cu at (143.9, 159.9)
- added R401: 1K, Resistor_SMD:R_0805_2012Metric, F.Cu at (153.7, 151.1)
- added R402: 4K7, Resistor_SMD:R_0805_2012Metric, F.Cu at (157.4, 173.5)
- added R403: 120, Resistor_SMD:R_0805_2012Metric, F.Cu at (153.3, 173.5)
- added R404: 4K7, Resistor_SMD:R_0805_2012Metric, F.Cu at (154.1, 159.9)
- added R501: 1K, Resistor_SMD:R_0805_2012Metric, F.Cu at (163.8, 151.1)
- added R502: 4K7, Resistor_SMD:R_0805_2012Metric, F.Cu at (167.5, 173.5)
- added R503: 120, Resistor_SMD:R_0805_2012Metric, F.Cu at (163.5, 173.5)
- added R504: 4K7, Resistor_SMD:R_0805_2012Metric, F.Cu at (164.2, 159.9)
- added R601: 1K, Resistor_SMD:R_0805_2012Metric, F.Cu at (174.0, 151.1)
- added R602: 4K7, Resistor_SMD:R_0805_2012Metric, F.Cu at (177.7, 173.5)
- added R603: 120, Resistor_SMD:R_0805_2012Metric, F.Cu at (173.6, 173.5)
- added R604: 4K7, Resistor_SMD:R_0805_2012Metric, F.Cu at (174.4, 159.9)
- added U201: shiftregister_74HC595, Package_SO:SOP-16_3.9x9.9mm_P1.27mm, F.Cu at (133.8, 140.3)
- added U301: SP3485EN-L/TR, Package_SO:SOIC-8_3.9x4.9mm_P1.27mm, F.Cu at (145.7, 155.2)
- added U401: SP3485EN-L/TR, Package_SO:SOIC-8_3.9x4.9mm_P1.27mm, F.Cu at (155.8, 155.2)
- added U501: SP3485EN-L/TR, Package_SO:SOIC-8_3.9x4.9mm_P1.27mm, F.Cu at (166.0, 155.2)
- added U601: SP3485EN-L/TR, Package_SO:SOIC-8_3.9x4.9mm_P1.27mm, F.Cu at (176.2, 155.2)
Routing:
- net +3V3: track 0.00 -> 55.8 mm
- net MODBUS_DI: track 0.00 -> 44.3 mm, vias 0 -> 4
- net /Hausreihe D/Haus S/B: track 0.00 -> 28.2 mm
- net /Hausreihe D/Haus T/B: track 0.00 -> 28.2 mm
- net /Hausreihe D/Haus R/B: track 0.00 -> 27.9 mm
- net /Hausreihe D/Haus U/B: track 0.00 -> 27.9 mm
- net /Hausreihe D/Haus U/A: track 0.00 -> 27.2 mm
- net /Hausreihe D/Haus S/A: track 0.00 -> 27.1 mm
- net /Hausreihe D/Haus R/A: track 0.00 -> 27.1 mm
- net /Hausreihe D/Haus T/A: track 0.00 -> 27.1 mm
- net GND: track 10.8 -> 25.2 mm, vias 0 -> 16
- net MODBUS_RO: track 0.00 -> 9.89 mm, vias 0 -> 4
- net /Hausreihe D/Haus T/ENABLE: track 0.00 -> 7.55 mm
- net /Hausreihe D/Haus S/ENABLE: track 0.00 -> 7.55 mm
- net /Hausreihe D/Haus R/ENABLE: track 0.00 -> 7.55 mm
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Other:
- board text removed: "${TITLE} ${ISSUE_DATE} v${REVISION}"

Commit message: Nach Review
Parts:
- added D304: SMAJ6.5CA, Diode_SMD:D_SMA, F.Cu at (199.4, 163.8)
- added D305: SMAJ6.5CA, Diode_SMD:D_SMA, F.Cu at (199.4, 168.3)
- added D404: SMAJ6.5CA, Diode_SMD:D_SMA, F.Cu at (219.4, 163.8)
- added D405: SMAJ6.5CA, Diode_SMD:D_SMA, F.Cu at (219.4, 168.3)
- added D504: SMAJ6.5CA, Diode_SMD:D_SMA, F.Cu at (239.4, 163.8)
- added D505: SMAJ6.5CA, Diode_SMD:D_SMA, F.Cu at (239.4, 168.3)
- added D604: SMAJ6.5CA, Diode_SMD:D_SMA, F.Cu at (259.4, 163.8)
- added D605: SMAJ6.5CA, Diode_SMD:D_SMA, F.Cu at (259.4, 168.3)
- added R305: 4K7, Resistor_SMD:R_0805_2012Metric, F.Cu at (193.1, 170.2)
- added R405: 4K7, Resistor_SMD:R_0805_2012Metric, F.Cu at (213.1, 170.2)
- added R505: 4K7, Resistor_SMD:R_0805_2012Metric, F.Cu at (233.1, 170.2)
- added R605: 4K7, Resistor_SMD:R_0805_2012Metric, F.Cu at (253.1, 170.2)
- D301, D401, D501, D601: value SMAJ6.5CA -> LED GREEN; footprint Diode_SMD:D_SMA -> 00_project_library:LED_0603_1608Metric
- D302, D402, D502, D602: value SMAJ6.5CA -> LED WHITE; footprint Diode_SMD:D_SMA -> 00_project_library:LED_0603_1608Metric
- R301, R401, R501, R601: value 1K -> 470
- R302, R402, R502, R602: value 4K7 -> 470
- R303, R403, R503, R603: value 120 -> 4K7
- R304, R404, R504, R604: value 4K7 -> 120
- moved H101 214.0 mm to (120.4, 211.1)
- moved H103 214.0 mm to (120.4, 227.0)
- moved H104 214.0 mm to (120.4, 235.0)
- moved H102 214.0 mm to (120.4, 219.1)
- moved J101 134.7 mm to (142.8, 202.6)
- moved D603 86.7 mm to (259.4, 159.2), turned to 0 degrees
- moved D602 86.1 mm to (261.4, 175.6)
- moved D601 82.7 mm to (261.4, 173.0), turned to 0 degrees
- moved U601 81.4 mm to (255.1, 174.9)
- moved Haus201 80.6 mm to (117.1, 180.1), turned to 0 degrees
- moved R603 80.0 mm to (253.1, 164.3), turned to 0 degrees
- moved R601 79.4 mm to (253.1, 158.4), turned to 0 degrees
- moved R604 79.1 mm to (253.1, 167.3), turned to 0 degrees
- moved D503 76.9 mm to (239.4, 159.2), turned to 0 degrees
- moved R602 76.4 mm to (253.1, 161.4), turned to 0 degrees
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Connections:
- D301 pad 1: /Hausreihe D/Haus R/A -> Net-(D301-K)
- D301 pad 2: GND -> +3V3
- D302 pad 1: /Hausreihe D/Haus R/B -> Net-(D302-K)
- D302 pad 2: /Hausreihe D/Haus R/A -> /Hausreihe D/Haus R/MODBUS_DE
- D303 pad 1: GND -> /Hausreihe D/Haus R/A
- D303 pad 2: /Hausreihe D/Haus R/B -> GND
- D401 pad 1: /Hausreihe D/Haus S/A -> Net-(D401-K)
- D401 pad 2: GND -> +3V3
- D402 pad 1: /Hausreihe D/Haus S/B -> Net-(D402-K)
- D402 pad 2: /Hausreihe D/Haus S/A -> /Hausreihe D/Haus S/MODBUS_DE
- D403 pad 1: GND -> /Hausreihe D/Haus S/A
- D403 pad 2: /Hausreihe D/Haus S/B -> GND
- D501 pad 1: /Hausreihe D/Haus T/A -> Net-(D501-K)
- D501 pad 2: GND -> +3V3
- D502 pad 1: /Hausreihe D/Haus T/B -> Net-(D502-K)
- D502 pad 2: /Hausreihe D/Haus T/A -> /Hausreihe D/Haus T/MODBUS_DE
- D503 pad 1: GND -> /Hausreihe D/Haus T/A
- D503 pad 2: /Hausreihe D/Haus T/B -> GND
- D601 pad 1: /Hausreihe D/Haus U/A -> Net-(D601-K)
- D601 pad 2: GND -> +3V3
- D602 pad 1: /Hausreihe D/Haus U/B -> Net-(D602-K)
- D602 pad 2: /Hausreihe D/Haus U/A -> /Hausreihe D/Haus U/MODBUS_DE
- D603 pad 1: GND -> /Hausreihe D/Haus U/A
- D603 pad 2: /Hausreihe D/Haus U/B -> GND
- J201 pad 10: /Hausreihe D/Haus T/B -> unconnected-(J201-Pad10)
- J201 pad 11: /Hausreihe D/Haus U/A -> unconnected-(J201-Pad11)
- J201 pad 12: /Hausreihe D/Haus U/B -> unconnected-(J201-Pad12)
- J201 pad 8: /Hausreihe D/Haus S/B -> unconnected-(J201-Pad8)
- J201 pad 9: /Hausreihe D/Haus T/A -> unconnected-(J201-Pad9)
- R301 pad 1: MODBUS_RO -> Net-(D301-K)
- R301 pad 2: Net-(U301-RO) -> /Hausreihe D/Haus R/MODBUS_RE
- R302 pad 1: GND -> Net-(D302-K)
- R302 pad 2: /Hausreihe D/Haus R/A -> GND
- R303 pad 1: /Hausreihe D/Haus R/A -> GND
- R303 pad 2: /Hausreihe D/Haus R/B -> /Hausreihe D/Haus R/A
- R304 pad 1: /Hausreihe D/Haus R/B -> /Hausreihe D/Haus R/A
- R304 pad 2: +3V3 -> /Hausreihe D/Haus R/B
- R401 pad 1: MODBUS_RO -> Net-(D401-K)
- R401 pad 2: Net-(U401-RO) -> /Hausreihe D/Haus S/MODBUS_RE
- R402 pad 1: GND -> Net-(D402-K)
- R402 pad 2: /Hausreihe D/Haus S/A -> GND
- R403 pad 1: /Hausreihe D/Haus S/A -> GND
- R403 pad 2: /Hausreihe D/Haus S/B -> /Hausreihe D/Haus S/A
- R404 pad 1: /Hausreihe D/Haus S/B -> /Hausreihe D/Haus S/A
- R404 pad 2: +3V3 -> /Hausreihe D/Haus S/B
- R501 pad 1: MODBUS_RO -> Net-(D501-K)
- R501 pad 2: Net-(U501-RO) -> /Hausreihe D/Haus T/MODBUS_RE
- R502 pad 1: GND -> Net-(D502-K)
- R502 pad 2: /Hausreihe D/Haus T/A -> GND
- R503 pad 1: /Hausreihe D/Haus T/A -> GND
- R503 pad 2: /Hausreihe D/Haus T/B -> /Hausreihe D/Haus T/A
- R504 pad 1: /Hausreihe D/Haus T/B -> /Hausreihe D/Haus T/A
- R504 pad 2: +3V3 -> /Hausreihe D/Haus T/B
- R601 pad 1: MODBUS_RO -> Net-(D601-K)
- R601 pad 2: Net-(U601-RO) -> /Hausreihe D/Haus U/MODBUS_RE
- R602 pad 1: GND -> Net-(D602-K)
- R602 pad 2: /Hausreihe D/Haus U/A -> GND
- R603 pad 1: /Hausreihe D/Haus U/A -> GND
- R603 pad 2: /Hausreihe D/Haus U/B -> /Hausreihe D/Haus U/A
- R604 pad 1: /Hausreihe D/Haus U/B -> /Hausreihe D/Haus U/A
- R604 pad 2: +3V3 -> /Hausreihe D/Haus U/B
- U201 pad 1: /Hausreihe D/Haus S/ENABLE -> /Hausreihe D/Haus R/MODBUS_DE
- U201 pad 15: /Hausreihe D/Haus R/ENABLE -> /Hausreihe D/Haus R/MODBUS_RE
- U201 pad 2: /Hausreihe D/Haus T/ENABLE -> unconnected-(U201-QC-Pad2)
- U201 pad 3: /Hausreihe D/Haus U/ENABLE -> unconnected-(U201-QD-Pad3)
- U301 pad 1: Net-(U301-RO) -> MODBUS_RO
- U301 pad 2: /Hausreihe D/Haus R/ENABLE -> /Hausreihe D/Haus R/MODBUS_RE
- U301 pad 3: /Hausreihe D/Haus R/ENABLE -> /Hausreihe D/Haus R/MODBUS_DE
- U401 pad 1: Net-(U401-RO) -> MODBUS_RO
- U401 pad 2: /Hausreihe D/Haus S/ENABLE -> /Hausreihe D/Haus S/MODBUS_RE
- U401 pad 3: /Hausreihe D/Haus S/ENABLE -> /Hausreihe D/Haus S/MODBUS_DE
- U501 pad 1: Net-(U501-RO) -> MODBUS_RO
- U501 pad 2: /Hausreihe D/Haus T/ENABLE -> /Hausreihe D/Haus T/MODBUS_RE
- U501 pad 3: /Hausreihe D/Haus T/ENABLE -> /Hausreihe D/Haus T/MODBUS_DE
- U601 pad 1: Net-(U601-RO) -> MODBUS_RO
- U601 pad 2: /Hausreihe D/Haus U/ENABLE -> /Hausreihe D/Haus U/MODBUS_RE
- U601 pad 3: /Hausreihe D/Haus U/ENABLE -> /Hausreihe D/Haus U/MODBUS_DE
Routing:
- net +3V3: track 55.8 -> 0.00 mm
- net MODBUS_DI: track 44.3 -> 0.00 mm, vias 4 -> 0
- net /Hausreihe D/Haus S/B: track 28.2 -> 0.00 mm
- net /Hausreihe D/Haus T/B: track 28.2 -> 0.00 mm
- net /Hausreihe D/Haus R/B: track 27.9 -> 0.00 mm
- net /Hausreihe D/Haus U/B: track 27.9 -> 0.00 mm
- net /Hausreihe D/Haus U/A: track 27.2 -> 0.00 mm
- net /Hausreihe D/Haus S/A: track 27.1 -> 0.00 mm
- net /Hausreihe D/Haus R/A: track 27.1 -> 0.00 mm
- net /Hausreihe D/Haus T/A: track 27.1 -> 0.00 mm
- net GND: track 25.2 -> 0.00 mm, vias 16 -> 0
- net MODBUS_RO: track 9.89 -> 0.00 mm, vias 4 -> 0
- net /Hausreihe D/Haus T/ENABLE: track 7.55 -> 0.00 mm
- net /Hausreihe D/Haus S/ENABLE: track 7.55 -> 0.00 mm
- net /Hausreihe D/Haus R/ENABLE: track 7.55 -> 0.00 mm
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- removed copper zone on B.Cu, net GND
- removed copper zone on F.Cu, net GND
