File: steuerung_automatik/hardware/pcb_kicad/pcb_zentral_pi.kicad_sch (KiCad schematic)
At the start: 40 parts, among them J1 USB_C_Receptacle_USB2.0, J2 weidmueller_SL 5.08HC-04-180, J3 weidmueller_SL 5.08HC-12-180, SW1 SW_MEC_5E, SW2 SW_MEC_5E, U1 RP2040, U2 W25Q128JVS, U3 AMS1117-3.3, U4 SP3485EN-L/TR, Y1 Crystal_GND24_Small

Commit message: Vor Review
Parts:
- removed C1, C10, C11, C12, C13, C14, C2, C5, C6, C9: 100n, Capacitor_SMD:C_0402_1005Metric_Pad0.74x0.62mm_HandSolder, symbol 00_project_library:C
- removed C15, C16: 10u, Capacitor_SMD:C_0603_1608Metric, symbol 00_project_library:C
- removed C3, C4: 1u, Capacitor_SMD:C_0402_1005Metric_Pad0.74x0.62mm_HandSolder, symbol 00_project_library:C
- removed C7, C8: 30p, Capacitor_SMD:C_0402_1005Metric, symbol 00_project_library:C
- removed D1: LED GREEN, 00_project_library:LED_0603_1608Metric, symbol 00_project_library:LED GREEN
- removed J1: USB_C_Receptacle_USB2.0, 00_project_library:USB_C_Receptacle_Palconn_UTC16-G, symbol 00_project_library:USB_C_Receptacle_USB2.0
- removed J2: weidmueller_SL 5.08HC-04-180, 00_project_library:weidmueller_SL 5.08HC-04-180, symbol 00_project_library:weidmueller_SL 5.08HC-04-180
- removed J3: weidmueller_SL 5.08HC-12-180, 00_project_library:weidmueller_SL 5.08HC-12-180, symbol 00_project_library:weidmueller_SL 5.08HC-12-180
- removed R1, R2: 5.1K, Resistor_SMD:R_0402_1005Metric_Pad0.72x0.64mm_HandSolder, symbol Device:R
- removed R3, R4: 27R, Resistor_SMD:R_0402_1005Metric_Pad0.72x0.64mm_HandSolder, symbol Device:R
- removed R5, R7: 10K, Resistor_SMD:R_0402_1005Metric_Pad0.72x0.64mm_HandSolder, symbol Device:R
- removed R6: 470R, Resistor_SMD:R_0402_1005Metric_Pad0.72x0.64mm_HandSolder, symbol Device:R
- removed R8: 1k, Resistor_SMD:R_0402_1005Metric_Pad0.72x0.64mm_HandSolder, symbol Device:R
- removed SW1, SW2: SW_MEC_5E, 00_project_library:SW_TS-1187A-B-A-B, symbol 00_project_library:SW_MEC_5E
- removed TP1: TestPoint, TestPoint:TestPoint_Pad_D2.5mm, symbol Connector:TestPoint
- removed U1: RP2040, 00_project_library:RP2040-QFN-56, symbol 00_project_library:RP2040
- removed U2: W25Q128JVS, 00_project_library:SOIC-8_5.23x5.23mm_P1.27mm, symbol 00_project_library:W25Q128JVS
- removed U3: AMS1117-3.3, 00_project_library:SOT-223-3_TabPin2, symbol 00_project_library:AMS1117-3.3
- removed U4: SP3485EN-L/TR, Package_SO:SOIC-8_3.9x4.9mm_P1.27mm, symbol 00_project_library:modbus_SP3485EN
- removed Y1: Crystal_GND24_Small, 00_project_library:Crystal_SMD_3225-4Pin_3.2x2.5mm, symbol 00_project_library:Crystal_GND24_Small
- added J101: pi_zero, 00_project_library:rpi_zero_bottom, symbol 00_project_library:pi_zero
- renumbered H1 to H101, H2 to H102, H3 to H103, H4 to H104
Connections:
- new net Hausreihe D/BIT_IN: J101.12 (GPIO18)
- new net MODBUS_DI: J101.10 (GPIO15_RXD0)
- new net MODBUS_RO: J101.8 (GPIO14_TXD0)
- new net SHIFTREGISTER_CLOCK: J101.18 (GPIO24)
- new net SHIFTREGISTER_OE: J101.16 (GPIO23)
- no-connect marks 34 -> 0
Other:
- added sheet Hausreihe D (pcb_zentral_hausreihe.kicad_sch)
- note removed: "Bypass Capacitors"
- note removed: "C1, C2 = 2*CL - 2*Cs CL = 20pF, Cs can be ~5pF"
- note removed: "Crystal"
- note removed: "Flash Memory"
- note removed: "Main Regulator"
- note removed: "Make sure 27R are close to RP2040"
- note removed: "Place 1uF close to pin 44"
- note removed: "Place 1uF close to pin 45"
- note removed: "Power LED"
- note removed: "RP2040"
- note removed: "Reset"
- note removed: "USB Type-C"

Commit message: Nach Review
Other:
- added sheet Hausreihe E (pcb_zentral_hausreihe.kicad_sch)
Changed lines of the file:
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@@
+    (stroke (width 0) (type default))
+  )
+  (wire (pts (xy 224.028 64.516) (xy 224.028 71.882))
     (stroke (width 0) (type default))
   )
@@
       )
     )
+  )
+  (sheet (at 207.264 71.882) (size 36.068 18.288) (fields_autoplaced)
+    (stroke (width 0.1524) (type solid))
+    (fill (color 0 0 0 0.0000))
+    (property "Sheetname" "Hausreihe E" (at 207.264 71.1704 0)
+      (effects (font (size 1.27 1.27)) (justify left bottom))
+    )
+    (property "Sheetfile" "pcb_zentral_hausreihe.kicad_sch" (at 207.264 90.7546 0)
+      (effects (font (size 1.27 1.27)) (justify left top))
+    )
+    (pin "485_0V" input (at 207.264 84.328 180)
+      (effects (font (size 1.27 1.27)) (justify left))
+    )
+    (pin "485_24V" input (at 207.264 80.772 180)
+      (effects (font (size 1.27 1.27)) (justify left))
+    )
+    (pin "+3V3" input (at 207.264 75.438 180)
+      (effects (font (size 1.27 1.27)) (justify left))
+    )
+    (pin "BIT_OUT" input (at 224.282 90.17 270)
+      (effects (font (size 1.27 1.27)) (justify left))
+    )
+    (pin "BIT_IN" input (at 224.028 71.882 90)
+      (effects (font (size 1.27 1.27)) (justify right))
+    )
+    (instances
+      (project "pcb_zentral_pi"
+        (path "/35c47459-45a7-4753-acae-c8b47e7575e1" (page "7"))
+      )
+    )
