File: steuerung_automatik/hardware/pcb_kicad/pcb_dezentral.kicad_pcb (KiCad board)
At the start: 2 copper layers, 55 x 78 mm, 84 parts, among them J1 weidmueller_SL5.08HC-06-90, J2 weidmueller_SL5.08HC-10-90, J901 USB_C_Receptacle_USB2.0, Q1 AO3400A, SW1 dip_switch_SPST16, SW901 SW_MEC_5E, U1 SP3485EN-L/TR, U2 AOZ1282CI, U901 RP2040, U902 AMS1117-3.3, U903 W25Q128JVS, Y901 Crystal_GND24_Small

Commit message: Schema dezentral komplett
Parts:
- J1: value weidmueller_SL5.08HC-06-90 -> 1146810000
- moved C915 174.6 mm to (81.9, 98.7), turned to 90 degrees
- moved C914 174.2 mm to (81.1, 106.0), turned to 180 degrees
- moved C913 174.1 mm to (81.1, 104.7), turned to 180 degrees
- moved C907 169.9 mm to (83.0, 96.9), turned to 90 degrees
- moved C908 168.2 mm to (85.1, 96.6), turned to 180 degrees
- moved C905 166.4 mm to (84.6, 93.4), turned to 90 degrees
- moved C904 166.2 mm to (82.5, 108.0), turned to -90 degrees
- moved C916 163.0 mm to (92.7, 106.6)
- moved C912 162.8 mm to (88.8, 115.2)
- moved C903 161.9 mm to (86.6, 107.4), turned to -90 degrees
- moved C911 160.8 mm to (92.2, 101.8)
- moved R905 153.6 mm to (76.3, 120.4)
- moved C906 151.5 mm to (96.7, 118.6)
- moved R9 141.6 mm to (99.9, 116.6), turned to -90 degrees
- moved U1 140.2 mm to (106.3, 108.0)
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Connections:
- net 485_0V renamed GND
- C6 pad 2: ds_3V3 -> +3V3
- C902 pad 1: ds_3V3 -> +3V3
- C906 pad 1: ds_3V3 -> +3V3
- C907 pad 1: ds_3V3 -> +3V3
- C908 pad 1: ds_3V3 -> +3V3
- C911 pad 1: ds_3V3 -> +3V3
- C912 pad 1: ds_3V3 -> +3V3
- C913 pad 1: ds_3V3 -> +3V3
- C914 pad 1: ds_3V3 -> +3V3
- C915 pad 1: ds_3V3 -> +3V3
- C916 pad 1: ds_3V3 -> +3V3
- D1 pad 1: ds_3V3 -> +3V3
- D11 pad 1: ds_3V3 -> +3V3
- D13 pad 1: ds_3V3 -> +3V3
- D15 pad 1: ds_3V3 -> +3V3
- D3 pad 1: ds_3V3 -> +3V3
- D5 pad 1: ds_3V3 -> +3V3
- D7 pad 1: ds_3V3 -> +3V3
- D9 pad 1: ds_3V3 -> +3V3
- D901 pad 2: ds_3V3 -> +3V3
- J2 pad 9: ds_3V3 -> +3V3
- R1 pad 1: ds_3V3 -> +3V3
- R2 pad 1: ds_3V3 -> +3V3
- R3 pad 1: ds_3V3 -> +3V3
- R4 pad 1: ds_3V3 -> +3V3
- R5 pad 1: ds_3V3 -> +3V3
- R6 pad 1: ds_3V3 -> +3V3
- R7 pad 1: ds_3V3 -> +3V3
- R8 pad 1: ds_3V3 -> +3V3
- R907 pad 1: ds_3V3 -> +3V3
- SW1 pad 1-1: ds_3V3 -> +3V3
- SW1 pad 2-1: ds_3V3 -> +3V3
- SW1 pad 3-1: ds_3V3 -> +3V3
- SW1 pad 4-1: ds_3V3 -> +3V3
- SW1 pad 5-1: ds_3V3 -> +3V3
- SW1 pad 6-1: ds_3V3 -> +3V3
- SW1 pad 7-1: ds_3V3 -> +3V3
- SW1 pad 8-1: ds_3V3 -> +3V3
- U1 pad 8: +3.3V -> +3V3
- U901 pad 1: ds_3V3 -> +3V3
- U901 pad 10: ds_3V3 -> +3V3
- U901 pad 11: modbus_addr_0 -> modbus_addr_7
- U901 pad 12: modbus_addr_1 -> modbus_addr_6
- U901 pad 13: modbus_addr_2 -> modbus_addr_5
- U901 pad 14: modbus_addr_3 -> modbus_addr_4
- U901 pad 15: modbus_addr_4 -> modbus_addr_3
- U901 pad 16: modbus_addr_5 -> modbus_addr_2
- U901 pad 17: modbus_addr_6 -> modbus_addr_1
- U901 pad 18: modbus_addr_7 -> modbus_addr_0
- U901 pad 22: ds_3V3 -> +3V3
- U901 pad 26: /cpu/RUN -> +3V3
- U901 pad 33: ds_3V3 -> +3V3
- U901 pad 42: ds_3V3 -> +3V3
- U901 pad 43: ds_3V3 -> +3V3
- U901 pad 44: ds_3V3 -> +3V3
- U901 pad 48: ds_3V3 -> +3V3
- U901 pad 49: ds_3V3 -> +3V3
- U901 pad 5: unconnected-(U901-GPIO3-Pad5) -> rel
- U902 pad 2: ds_3V3 -> +3V3
- U903 pad 8: ds_3V3 -> +3V3
Routing:
- net +3V3: track 0.00 -> 282.2 mm, vias 0 -> 2
- net ds_3V3: track 223.2 -> 0.00 mm
- net rel: track 0.00 -> 44.2 mm, vias 0 -> 3
- net GND: track 55.7 -> 90.3 mm, vias 15 -> 45
- net 485_A: track 0.00 -> 33.7 mm
- net 485_24V: track 13.4 -> 38.5 mm
- net 485_B: track 0.00 -> 22.9 mm
- net +1V1: track 0.00 -> 22.7 mm, vias 0 -> 4
- net MODBUS_DE: track 0.00 -> 16.6 mm
- net MODBUS_DI: track 0.00 -> 16.0 mm
- net modbus_addr_0: track 0.00 -> 15.6 mm
- net MODBUS_RO: track 0.00 -> 14.6 mm, vias 0 -> 2
- net modbus_addr_1: track 0.00 -> 12.9 mm
- net rel_n: track 0.00 -> 11.6 mm
- net modbus_addr_2: track 0.00 -> 10.1 mm
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Other:
- board size 55 x 78 mm -> 55 x 73.5 mm

Commit message: Fix J12
Parts:
- J2: value weidmueller_SL5.08HC-10-90 -> 1146900000
Changed lines of the file:
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@@
         (effects (font (size 1.27 1.27) (thickness 0.254)))
     )
-    (fp_text value "weidmueller_SL5.08HC-10-90" (at -22.86 4) (layer "F.SilkS") hide
+    (fp_text value "1146900000" (at -22.86 4) (layer "F.SilkS") hide
         (effects (font (size 1.27 1.27) (thickness 0.254)))
     )
@@
     (pad "10" thru_hole circle (at -45.72 0 180) (size 1.95 1.95) (drill 1.3) (layers "*.Cu" "*.Mask")
       (net 8 "GND") (pinfunction "10") (pintype "passive"))
-    (model "/home/maerki/work_heizung/puenterswis_heizung_2023_git/steuerung_automatik/hardware/pcb_kicad/00_project_parts/weidmueller/1146900000/3D/1146900000.stp"
+    (model "${KIPRJMOD}/00_project_parts/weidmueller/1146900000/3D/1146900000.stp"
       (offset (xyz -48 -10 -3.24))
       (scale (xyz 1 1 1))
