File: steuerung_automatik/hardware/pcb_kicad/pcb_dezentral_cpu.kicad_sch (KiCad schematic)
At the start: 32 parts, among them J1 USB_C_Receptacle_USB2.0, SW2 SW_MEC_5E, U1 RP2040, U3 W25Q128JVS, U4 AMS1117-3.3, Y1 Crystal_GND24_Small

Commit message: Schema dezentral komplett
Connections:
- net RUN is gone; now on net +3V3: U1.26 (RUN)
- net modbus_addr_0: now also U1.18 (GPIO15); no longer U1.11 (GPIO8)
- net modbus_addr_1: now also U1.17 (GPIO14); no longer U1.12 (GPIO9)
- net modbus_addr_2: now also U1.16 (GPIO13); no longer U1.13 (GPIO10)
- net modbus_addr_3: now also U1.15 (GPIO12); no longer U1.14 (GPIO11)
- net modbus_addr_4: now also U1.14 (GPIO11); no longer U1.15 (GPIO12)
- net modbus_addr_5: now also U1.13 (GPIO10); no longer U1.16 (GPIO13)
- net modbus_addr_6: now also U1.12 (GPIO9); no longer U1.17 (GPIO14)
- net modbus_addr_7: now also U1.11 (GPIO8); no longer U1.18 (GPIO15)
- net rel: now reaches U1.5 (GPIO3)
- no-connect marks 9 -> 14
Changed lines of the file:
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@@
   (junction (at 189.992 70.358) (diameter 0) (color 0 0 0 0)
   )
+  (no_connect (at 43.942 95.504))
   (no_connect (at 176.276 100.838))
   (no_connect (at 43.942 52.324))
   (no_connect (at 176.276 98.298))
   (no_connect (at 115.062 52.324))
+  (no_connect (at 43.942 92.964))
+  (no_connect (at 43.942 90.424))
+  (no_connect (at 43.942 87.884))
+  (no_connect (at 115.062 54.864))
   (no_connect (at 43.942 54.864))
-  (no_connect (at 115.062 54.864))
-  (no_connect (at 43.942 49.784))
+  (no_connect (at 43.942 98.044))
+  (no_connect (at 43.942 100.584))
   (no_connect (at 43.942 59.944))
   (no_connect (at 43.942 57.404))
@@
     (stroke (width 0) (type solid))
   )
-  (wire (pts (xy 115.062 43.434) (xy 126.492 43.434))
+  (wire (pts (xy 115.062 43.434) (xy 118.364 43.434))
     (stroke (width 0) (type solid))
   )
@@
     (effects (font (size 1.27 1.27) italic) (justify right bottom))
   )
-  (label "RUN" (at 126.492 43.434 180) (fields_autoplaced)
-    (effects (font (size 1.27 1.27) italic) (justify right bottom))
-  )
   (label "XIN" (at 262.128 134.112 180) (fields_autoplaced)
     (effects (font (size 1.27 1.27) italic) (justify right bottom))
@@
     (effects (font (size 1.27 1.27) italic) (justify right bottom))
   )
-  (global_label "modbus_addr_1" (shape input) (at 43.942 67.564 180) (fields_autoplaced)
-    (effects (font (size 1.27 1.27)) (justify right))
-    (property "Intersheetrefs" "${INTERSHEET_REFS}" (at 26.1664 67.564 0)
+  (global_label "modbus_addr_5" (shape input) (at 43.942 70.104 180) (fields_autoplaced)
+    (effects (font (size 1.27 1.27)) (justify right))
+    (property "Intersheetrefs" "${INTERSHEET_REFS}" (at 26.1664 70.104 0)
+      (effects (font (size 1.27 1.27)) (justify right) hide)
+    )
+  )
+  (global_label "modbus_addr_4" (shape input) (at 43.942 72.644 180) (fields_autoplaced)
+    (effects (font (size 1.27 1.27)) (justify right))
+    (property "Intersheetrefs" "${INTERSHEET_REFS}" (at 26.1664 72.644 0)
       (effects (font (size 1.27 1.27)) (justify right) hide)
     )
@@
     )
   )
-  (global_label "modbus_addr_2" (shape input) (at 43.942 70.104 180) (fields_autoplaced)
-    (effects (font (size 1.27 1.27)) (justify right))
-    (property "Intersheetrefs" "${INTERSHEET_REFS}" (at 26.1664 70.104 0)
-      (effects (font (size 1.27 1.27)) (justify right) hide)
-    )
-  )
-  (global_label "modbus_addr_4" (shape input) (at 43.942 75.184 180) (fields_autoplaced)
-    (effects (font (size 1.27 1.27)) (justify right))
-    (property "Intersheetrefs" "${INTERSHEET_REFS}" (at 26.1664 75.184 0)
-      (effects (font (size 1.27 1.27)) (justify right) hide)
-    )
-  )
   (global_label "ds_7" (shape bidirectional) (at 43.942 103.124 180) (fields_autoplaced)
     (effects (font (size 1.27 1.27)) (justify right))
     (property "Intersheetrefs" "${INTERSHEET_REFS}" (at 35.4915 103.124 0)
+      (effects (font (size 1.27 1.27)) (justify right) hide)
+    )
+  )
+  (global_label "modbus_addr_2" (shape input) (at 43.942 77.724 180) (fields_autoplaced)
+    (effects (font (size 1.27 1.27)) (justify right))
+    (property "Intersheetrefs" "${INTERSHEET_REFS}" (at 26.1664 77.724 0)
       (effects (font (size 1.27 1.27)) (justify right) hide)
     )
@@
     )
   )
+  (global_label "modbus_addr_3" (shape input) (at 43.942 75.184 180) (fields_autoplaced)
+    (effects (font (size 1.27 1.27)) (justify right))
+    (property "Intersheetrefs" "${INTERSHEET_REFS}" (at 26.1664 75.184 0)
+      (effects (font (size 1.27 1.27)) (justify right) hide)
+    )
+  )
   (global_label "ds_2" (shape bidirectional) (at 115.062 98.044 0) (fields_autoplaced)
     (effects (font (size 1.27 1.27)) (justify left))
@@
     )
   )
-  (global_label "modbus_addr_0" (shape input) (at 43.942 65.024 180) (fields_autoplaced)
+  (global_label "rel" (shape output) (at 43.942 49.784 180) (fields_autoplaced)
+    (effects (font (size 1.27 1.27)) (justify right))
+    (property "Intersheetrefs" "${INTERSHEET_REFS}" (at 38.3217 49.784 0)
+      (effects (font (size 1.27 1.27)) (justify right) hide)
+    )
+  )
+  (global_label "ds_6" (shape bidirectional) (at 43.942 105.664 180) (fields_autoplaced)
+    (effects (font (size 1.27 1.27)) (justify right))
+    (property "Intersheetrefs" "${INTERSHEET_REFS}" (at 35.4915 105.664 0)
+      (effects (font (size 1.27 1.27)) (justify right) hide)
+    )
+  )
+  (global_label "MODBUS_RO" (shape input) (at 43.942 44.704 180) (fields_autoplaced)
+    (effects (font (size 1.27 1.27)) (justify right))
+    (property "Intersheetrefs" "${INTERSHEET_REFS}" (at 29.4317 44.704 0)
+      (effects (font (size 1.27 1.27)) (justify right) hide)
+    )
+  )
+  (global_label "modbus_addr_7" (shape input) (at 43.942 65.024 180) (fields_autoplaced)
     (effects (font (size 1.27 1.27)) (justify right))
     (property "Intersheetrefs" "${INTERSHEET_REFS}" (at 26.1664 65.024 0)
-      (effects (font (size 1.27 1.27)) (justify right) hide)
-    )
-  )
-  (global_label "modbus_addr_5" (shape input) (at 43.942 77.724 180) (fields_autoplaced)
-    (effects (font (size 1.27 1.27)) (justify right))
-    (property "Intersheetrefs" "${INTERSHEET_REFS}" (at 26.1664 77.724 0)
-      (effects (font (size 1.27 1.27)) (justify right) hide)
-    )
-  )
-  (global_label "ds_6" (shape bidirectional) (at 43.942 105.664 180) (fields_autoplaced)
-    (effects (font (size 1.27 1.27)) (justify right))
-    (property "Intersheetrefs" "${INTERSHEET_REFS}" (at 35.4915 105.664 0)
-      (effects (font (size 1.27 1.27)) (justify right) hide)
-    )
-  )
-  (global_label "MODBUS_RO" (shape input) (at 43.942 44.704 180) (fields_autoplaced)
-    (effects (font (size 1.27 1.27)) (justify right))
-    (property "Intersheetrefs" "${INTERSHEET_REFS}" (at 29.4317 44.704 0)
-      (effects (font (size 1.27 1.27)) (justify right) hide)
-    )
-  )
-  (global_label "modbus_addr_3" (shape input) (at 43.942 72.644 180) (fields_autoplaced)
-    (effects (font (size 1.27 1.27)) (justify right))
-    (property "Intersheetrefs" "${INTERSHEET_REFS}" (at 26.1664 72.644 0)
       (effects (font (size 1.27 1.27)) (justify right) hide)
     )
@@
     )
   )
-  (global_label "modbus_addr_7" (shape input) (at 43.942 82.804 180) (fields_autoplaced)
+  (global_label "modbus_addr_0" (shape input) (at 43.942 82.804 180) (fields_autoplaced)
     (effects (font (size 1.27 1.27)) (justify right))
     (property "Intersheetrefs" "${INTERSHEET_REFS}" (at 26.1664 82.804 0)
+      (effects (font (size 1.27 1.27)) (justify right) hide)
+    )
+  )
+  (global_label "modbus_addr_1" (shape input) (at 43.942 80.264 180) (fields_autoplaced)
+    (effects (font (size 1.27 1.27)) (justify right))
+    (property "Intersheetrefs" "${INTERSHEET_REFS}" (at 26.1664 80.264 0)
+      (effects (font (size 1.27 1.27)) (justify right) hide)
+    )
+  )
+  (global_label "modbus_addr_6" (shape input) (at 43.942 67.564 180) (fields_autoplaced)
+    (effects (font (size 1.27 1.27)) (justify right))
+    (property "Intersheetrefs" "${INTERSHEET_REFS}" (at 26.1664 67.564 0)
       (effects (font (size 1.27 1.27)) (justify right) hide)
     )
@@
     )
   )
-  (global_label "modbus_addr_6" (shape input) (at 43.942 80.264 180) (fields_autoplaced)
-    (effects (font (size 1.27 1.27)) (justify right))
-    (property "Intersheetrefs" "${INTERSHEET_REFS}" (at 26.1664 80.264 0)
-      (effects (font (size 1.27 1.27)) (justify right) hide)
-    )
-  )
   (symbol (lib_id "Device:R") (at 122.682 87.884 270) (unit 1)
     (in_bom yes) (on_board yes) (dnp no)
@@
         )
       )
+    )
+  )
+  (symbol (lib_id "power:+3V3") (at 118.364 43.434 270) (unit 1)
+    (in_bom yes) (on_board yes) (dnp no)
+    (property "Reference" "#PWR013" (at 114.554 43.434 0)
+      (effects (font (size 0.8 0.8)) hide)
+    )
+    (property "Value" "+3V3" (at 121.9962 43.307 0)
+      (effects (font (size 0.8 0.8)))
+    )
+    (property "Footprint" "" (at 118.364 43.434 0)
+      (effects (font (size 0.8 0.8)) hide)
+    )
+    (property "Datasheet" "" (at 118.364 43.434 0)
+      (effects (font (size 0.8 0.8)) hide)
+    )
+    (pin "1")
+    (instances
+      (project "pcb_dezentral"
+        (path "/35c47459-45a7-4753-acae-c8b47e7575e1"
+          (reference "#PWR013") (unit 1)
+        )
+        (path "/35c47459-45a7-4753-acae-c8b47e7575e1/24d7d496-8920-4421-a637-0c9bf263a085"
+          (reference "#PWR037") (unit 1)
+        )
+      )

Commit message: Anpassungen von Peter
Parts:
- added IO18, IO19, IO20: TestPoint, TestPoint:TestPoint_Pad_D1.0mm, symbol Connector:TestPoint
Connections:
- net at U1.29 (GPIO18): now also IO18.1
- net at U1.30 (GPIO19): now also IO19.1
- net at U1.31 (GPIO20): now also IO20.1
- net modbus_led: now reaches U1.32 (GPIO21)
- no-connect marks 14 -> 10
Changed lines of the file:
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@@
   (junction (at 189.992 70.358) (diameter 0) (color 0 0 0 0)
   )
-  (no_connect (at 43.942 95.504))
   (no_connect (at 176.276 100.838))
   (no_connect (at 43.942 52.324))
   (no_connect (at 176.276 98.298))
   (no_connect (at 115.062 52.324))
-  (no_connect (at 43.942 92.964))
   (no_connect (at 43.942 90.424))
   (no_connect (at 43.942 87.884))
   (no_connect (at 115.062 54.864))
   (no_connect (at 43.942 54.864))
-  (no_connect (at 43.942 98.044))
-  (no_connect (at 43.942 100.584))
   (no_connect (at 43.942 59.944))
   (no_connect (at 43.942 57.404))
@@
     (stroke (width 0) (type solid))
   )
+  (wire (pts (xy 41.148 98.044) (xy 43.942 98.044))
+    (stroke (width 0) (type default))
+  )
   (wire (pts (xy 214.63 100.076) (xy 214.63 96.266))
     (stroke (width 0) (type default))
@@
     (stroke (width 0) (type solid))
   )
+  (wire (pts (xy 41.148 95.504) (xy 43.942 95.504))
+    (stroke (width 0) (type default))
+  )
   (wire (pts (xy 244.348 144.272) (xy 249.428 144.272))
     (stroke (width 0) (type solid))
@@
     (stroke (width 0) (type solid))
   )
+  (wire (pts (xy 41.148 92.964) (xy 43.942 92.964))
+    (stroke (width 0) (type default))
+  )
   (wire (pts (xy 187.706 77.978) (xy 187.706 79.248))
     (stroke (width 0) (type solid))
@@
   (wire (pts (xy 177.546 88.138) (xy 187.706 88.138))
     (stroke (width 0) (type solid))
+  )
+  (wire (pts (xy 40.894 100.584) (xy 43.942 100.584))
+    (stroke (width 0) (type default))
   )
   (wire (pts (xy 189.992 70.358) (xy 191.77 70.358))
@@
     )
   )
+  (global_label "modbus_led" (shape output) (at 40.894 100.584 180) (fields_autoplaced)
+    (effects (font (size 1.27 1.27)) (justify right))
+    (property "Intersheetrefs" "${INTERSHEET_REFS}" (at 26.6259 100.584 0)
+      (effects (font (size 1.27 1.27)) (justify right) hide)
+    )
+  )
   (global_label "modbus_addr_2" (shape input) (at 43.942 77.724 180) (fields_autoplaced)
     (effects (font (size 1.27 1.27)) (justify right))
@@
         (path "/35c47459-45a7-4753-acae-c8b47e7575e1/24d7d496-8920-4421-a637-0c9bf263a085"
           (reference "R907") (unit 1)
+        )
+      )
+    )
+  )
+  (symbol (lib_id "Connector:TestPoint") (at 41.148 95.504 90) (unit 1)
+    (in_bom yes) (on_board yes) (dnp no)
+    (property "Reference" "IO19" (at 34.798 95.504 90)
+      (effects (font (size 1.27 1.27)))
+    )
+    (property "Value" "TestPoint" (at 37.846 92.964 90)
+      (effects (font (size 1.27 1.27)) hide)
+    )
+    (property "Footprint" "TestPoint:TestPoint_Pad_D1.0mm" (at 41.148 90.424 0)
+      (effects (font (size 1.27 1.27)) hide)
+    )
+    (property "Datasheet" "~" (at 41.148 90.424 0)
+      (effects (font (size 1.27 1.27)) hide)
+    )
+    (pin "1")
+    (instances
+      (project "pcb_dezentral"
+        (path "/35c47459-45a7-4753-acae-c8b47e7575e1/24d7d496-8920-4421-a637-0c9bf263a085"
+          (reference "IO19") (unit 1)
         )
       )
@@
     )
   )
+  (symbol (lib_id "Connector:TestPoint") (at 41.148 92.964 90) (unit 1)
+    (in_bom yes) (on_board yes) (dnp no)
+    (property "Reference" "IO18" (at 34.798 92.964 90)
+      (effects (font (size 1.27 1.27)))
+    )
+    (property "Value" "TestPoint" (at 37.846 90.424 90)
+      (effects (font (size 1.27 1.27)) hide)
+    )
+    (property "Footprint" "TestPoint:TestPoint_Pad_D1.0mm" (at 41.148 87.884 0)
+      (effects (font (size 1.27 1.27)) hide)
+    )
+    (property "Datasheet" "~" (at 41.148 87.884 0)
+      (effects (font (size 1.27 1.27)) hide)
+    )
+    (pin "1")
+    (instances
+      (project "pcb_dezentral"
+        (path "/35c47459-45a7-4753-acae-c8b47e7575e1/24d7d496-8920-4421-a637-0c9bf263a085"
+          (reference "IO18") (unit 1)
+        )
+      )
+    )
+  )
   (symbol (lib_id "00_project_library:C") (at 199.136 36.322 0) (unit 1)
     (in_bom yes) (on_board yes) (dnp no)
@@
         )
       )
+    )
+  )
+  (symbol (lib_id "Connector:TestPoint") (at 41.148 98.044 90) (unit 1)
+    (in_bom yes) (on_board yes) (dnp no)
+    (property "Reference" "IO20" (at 34.798 98.044 90)
+      (effects (font (size 1.27 1.27)))
+    )
+    (property "Value" "TestPoint" (at 37.846 95.504 90)
+      (effects (font (size 1.27 1.27)) hide)
+    )
+    (property "Footprint" "TestPoint:TestPoint_Pad_D1.0mm" (at 41.148 92.964 0)
+      (effects (font (size 1.27 1.27)) hide)
+    )
+    (property "Datasheet" "~" (at 41.148 92.964 0)
+      (effects (font (size 1.27 1.27)) hide)
+    )
+    (pin "1")
+    (instances
+      (project "pcb_dezentral"
+        (path "/35c47459-45a7-4753-acae-c8b47e7575e1/24d7d496-8920-4421-a637-0c9bf263a085"
+          (reference "IO20") (unit 1)
+        )
+      )

Commit message: pcb_dezentral v0.8
Connections:
- net modbus_led: no longer names the net of U1.32 (GPIO21)
- no-connect marks 10 -> 11
Changed lines of the file:
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@@
   (no_connect (at 176.276 98.298))
   (no_connect (at 115.062 52.324))
+  (no_connect (at 43.942 100.584))
   (no_connect (at 43.942 90.424))
   (no_connect (at 43.942 87.884))
@@
     (stroke (width 0) (type solid))
   )
-  (wire (pts (xy 40.894 100.584) (xy 43.942 100.584))
-    (stroke (width 0) (type default))
-  )
   (wire (pts (xy 189.992 70.358) (xy 191.77 70.358))
     (stroke (width 0) (type default))
@@
       (effects (font (size 1.27 1.27)) (justify right) hide)
     )
-  )
-  (global_label "modbus_led" (shape output) (at 40.894 100.584 180) (fields_autoplaced)
-    (effects (font (size 1.27 1.27)) (justify right))
-    (property "Intersheetrefs" "${INTERSHEET_REFS}" (at 26.6259 100.584 0)
-      (effects (font (size 1.27 1.27)) (justify right) hide)
-    )
