File: steuerung_automatik/hardware/pcb_kicad/pcb_dezentral.kicad_sch (KiCad schematic)
At the start: 57 parts, among them J1 weidmueller_SL5.08HC-06-90, J2 weidmueller_SL5.08HC-10-90, Q1 AO3400A, SW1 dip_switch_SPST16, U1 SP3485EN-L/TR, U2 AOZ1282CI

Commit message: pcb_dezentral v1.0
Parts:
- added C7: 100n 50V, Diode_SMD:D_0805_2012Metric, symbol Device:C
- added D28: LED WHITE, 00_project_library:LED_0603_1608Metric, symbol 00_project_library:LED WHITE
- added R17: 4k7, Resistor_SMD:R_0402_1005Metric_Pad0.72x0.64mm_HandSolder, symbol Device:R
- added R18, R19: 10k, Resistor_SMD:R_0402_1005Metric_Pad0.72x0.64mm_HandSolder, symbol Device:R
- added R20: 470R, Resistor_SMD:R_0402_1005Metric_Pad0.72x0.64mm_HandSolder, symbol Device:R
Connections:
- net +5V: now also R18.1
- net GND: now also R19.2, R20.1
- net 485_A renamed 485_D+
- net 485_D+: now also C7.2, R18.2
- net 485_B renamed 485_D-
- net 485_D-: now also R17.2, R19.1
- new net: C7.1, R17.1
- new net: D28.1 (K), R20.2
- new net ZENTRALE_LED: D28.2 (A)
Other:
- note added: "Biasing"
- note added: "Zentrale LED"
- moved on the sheet: C6, D1, D10, D11, D12, D13, D14, D15, D16, D17, D18, D2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
